Commit message: Smooth mode switching

File: morphobot-ros2/eternalmorph_description/urdf/eternalmorph.xacro (robot description, xacro)
@@ -124,7 +124,7 @@
   </visual>
   <collision>
-    <origin xyz="-0.293181 -0.244976 -0.019994" rpy="0 0 0"/>
-    <geometry>
-      <mesh filename="package://eternalmorph_description/meshes/sol_on_teker_1.stl" scale="0.001 0.001 0.001"/>
+    <origin xyz="-0.0165 0 0" rpy="0 1.5707963 0"/>
+    <geometry>
+      <cylinder radius="0.0795" length="0.033"/>
     </geometry>
   </collision>
@@ -144,7 +144,7 @@
   </visual>
   <collision>
-    <origin xyz="-0.293181 0.374976 -0.020006" rpy="0 0 0"/>
-    <geometry>
-      <mesh filename="package://eternalmorph_description/meshes/sol_arka_teker_1.stl" scale="0.001 0.001 0.001"/>
+    <origin xyz="-0.0165 0 0" rpy="0 1.5707963 0"/>
+    <geometry>
+      <cylinder radius="0.0795" length="0.033"/>
     </geometry>
   </collision>
@@ -164,7 +164,7 @@
   </visual>
   <collision>
-    <origin xyz="-0.546819 -0.244976 -0.020006" rpy="0 0 0"/>
-    <geometry>
-      <mesh filename="package://eternalmorph_description/meshes/sag_on_teker_1.stl" scale="0.001 0.001 0.001"/>
+    <origin xyz="0.0165 0 0" rpy="0 1.5707963 0"/>
+    <geometry>
+      <cylinder radius="0.0795" length="0.033"/>
     </geometry>
   </collision>
@@ -184,7 +184,7 @@
   </visual>
   <collision>
-    <origin xyz="-0.546819 0.374976 -0.019994" rpy="0 0 0"/>
-    <geometry>
-      <mesh filename="package://eternalmorph_description/meshes/sag_arka_teker_1.stl" scale="0.001 0.001 0.001"/>
+    <origin xyz="0.0165 0 0" rpy="0 1.5707963 0"/>
+    <geometry>
+      <cylinder radius="0.0795" length="0.033"/>
     </geometry>
   </collision>
@@ -475,4 +475,5 @@
   <child link="sol_on_teker_1"/>
   <axis xyz="1.0 0.0 0.0"/>
+  <dynamics damping="0.05" friction="0.01"/>
 </joint>
 <joint name="sol_arka_teker" type="continuous">
@@ -481,4 +482,5 @@
   <child link="sol_arka_teker_1"/>
   <axis xyz="1.0 0.0 0.0"/>
+  <dynamics damping="0.05" friction="0.01"/>
 </joint>
 <joint name="sag_on_teker" type="continuous">
@@ -487,4 +489,5 @@
   <child link="sag_on_teker_1"/>
   <axis xyz="1.0 0.0 0.0"/>
+  <dynamics damping="0.05" friction="0.01"/>
 </joint>
 <joint name="sag_arka_teker" type="continuous">
@@ -493,4 +496,5 @@
   <child link="sag_arka_teker_1"/>
   <axis xyz="1.0 0.0 0.0"/>
+  <dynamics damping="0.05" friction="0.01"/>
 </joint>
 <joint name="sol_on_pervane_joint" type="continuous">
@@ -528,5 +532,5 @@
   <child link="sol_on_tekerlek_eksen_1"/>
   <axis xyz="-1.0 -0.0 0.0"/>
-  <limit upper="1.570796" lower="-0.1" effort="200" velocity="100"/>
+  <limit upper="1.7" lower="-0.2" effort="200" velocity="100"/>
   <dynamics damping="2.0" friction="0.2"/>
 </joint>
@@ -536,5 +540,5 @@
   <child link="sol_on_tutucu_parca_1"/>
   <axis xyz="0.0 -1.0 -0.0"/>
-  <limit upper="0.1" lower="-1.570796" effort="200" velocity="100"/>
+  <limit upper="0.2" lower="-1.7" effort="200" velocity="100"/>
   <dynamics damping="2.0" friction="0.2"/>
 </joint>
@@ -544,5 +548,5 @@
   <child link="sag_on_tekerlek_eksen_1"/>
   <axis xyz="1.0 0.0 0.0"/>
-  <limit upper="0.1" lower="-1.570796" effort="200" velocity="100"/>
+  <limit upper="0.2" lower="-1.7" effort="200" velocity="100"/>
   <dynamics damping="2.0" friction="0.2"/>
 </joint>
@@ -552,5 +556,5 @@
   <child link="sag_on_tutucu_parca_1"/>
   <axis xyz="0.0 -1.0 0.0"/>
-  <limit upper="1.570796" lower="-0.1" effort="200" velocity="100"/>
+  <limit upper="1.7" lower="-0.2" effort="200" velocity="100"/>
   <dynamics damping="2.0" friction="0.2"/>
 </joint>
@@ -560,5 +564,5 @@
   <child link="sol_arka_tekerlek_eksen_1"/>
   <axis xyz="-1.0 -0.0 -0.0"/>
-  <limit upper="0.1" lower="-1.570796" effort="200" velocity="100"/>
+  <limit upper="0.2" lower="-1.7" effort="200" velocity="100"/>
   <dynamics damping="2.0" friction="0.2"/>
 </joint>
@@ -568,5 +572,5 @@
   <child link="sol_arka_tutucu_parca_1"/>
   <axis xyz="-0.0 1.0 0.0"/>
-  <limit upper="1.570796" lower="-0.1" effort="200" velocity="100"/>
+  <limit upper="1.7" lower="-0.2" effort="200" velocity="100"/>
   <dynamics damping="2.0" friction="0.2"/>
 </joint>
@@ -576,5 +580,5 @@
   <child link="sag_arka_tekerlek_eksen_1"/>
   <axis xyz="1.0 0.0 0.0"/>
-  <limit upper="1.570796" lower="-0.1" effort="200" velocity="100"/>
+  <limit upper="1.7" lower="-0.2" effort="200" velocity="100"/>
   <dynamics damping="2.0" friction="0.2"/>
 </joint>
@@ -584,5 +588,5 @@
   <child link="sag_arka_tutucu_parca_1"/>
   <axis xyz="-0.0 1.0 0.0"/>
-  <limit upper="0.1" lower="-1.570796" effort="200" velocity="100"/>
+  <limit upper="0.2" lower="-1.7" effort="200" velocity="100"/>
   <dynamics damping="2.0" friction="0.2"/>
 </joint>

Commit message: Fix propeller

File: morphobot-ros2/eternalmorph_description/urdf/eternalmorph.xacro (robot description, xacro)
@@ -352,10 +352,10 @@
 <link name="sol_on_pervane_1">
   <inertial>
-    <origin xyz="-0.0027102891123487183 -3.060681447453195e-07 2.643057327444964e-07" rpy="0 0 0"/>
+    <origin xyz="2.6430573e-07 -3.0606814e-07 0.0027102891" rpy="0 1.57079632679 0"/>
     <mass value="0.027453359988130525"/>
     <inertia ixx="1.0e-05" iyy="1e-05" izz="1e-05" ixy="-0.0" iyz="-0.0" ixz="-0.0"/>
   </inertial>
   <visual>
-    <origin xyz="-0.274181 -0.244976 -0.019994" rpy="0 0 0"/>
+    <origin xyz="-0.019994 -0.244976 0.274181" rpy="0 1.57079632679 0"/>
     <geometry>
       <mesh filename="package://eternalmorph_description/meshes/sol_on_pervane_1.stl" scale="0.001 0.001 0.001"/>
@@ -364,5 +364,5 @@
   </visual>
   <collision>
-    <origin xyz="-0.274181 -0.244976 -0.019994" rpy="0 0 0"/>
+    <origin xyz="-0.019994 -0.244976 0.274181" rpy="0 1.57079632679 0"/>
     <geometry>
       <mesh filename="package://eternalmorph_description/meshes/sol_on_pervane_1.stl" scale="0.001 0.001 0.001"/>
@@ -372,10 +372,10 @@
 <link name="sol_arka_pervane_1">
   <inertial>
-    <origin xyz="-0.0027102891123494954 5.542049622553336e-07 -1.1353977304173757e-07" rpy="0 0 0"/>
+    <origin xyz="-1.1353977e-07 5.5420496e-07 0.0027102891" rpy="0 1.57079632679 0"/>
     <mass value="0.027453359988130525"/>
     <inertia ixx="1.0e-05" iyy="1e-05" izz="1e-05" ixy="-0.0" iyz="-0.0" ixz="-0.0"/>
   </inertial>
   <visual>
-    <origin xyz="-0.274181 0.374976 -0.019614" rpy="0 0 0"/>
+    <origin xyz="-0.019614 0.374976 0.274181" rpy="0 1.57079632679 0"/>
     <geometry>
       <mesh filename="package://eternalmorph_description/meshes/sol_arka_pervane_1.stl" scale="0.001 0.001 0.001"/>
@@ -384,5 +384,5 @@
   </visual>
   <collision>
-    <origin xyz="-0.274181 0.374976 -0.019614" rpy="0 0 0"/>
+    <origin xyz="-0.019614 0.374976 0.274181" rpy="0 1.57079632679 0"/>
     <geometry>
       <mesh filename="package://eternalmorph_description/meshes/sol_arka_pervane_1.stl" scale="0.001 0.001 0.001"/>
@@ -392,10 +392,10 @@
 <link name="sag_arka_pervane_1">
   <inertial>
-    <origin xyz="0.0027102891123486073 -3.04781677812338e-07 1.4261012662442063e-07" rpy="0 0 0"/>
+    <origin xyz="-1.4261013e-07 -3.0478168e-07 0.0027102891" rpy="0 -1.57079632679 0"/>
     <mass value="0.027453359988130525"/>
     <inertia ixx="1.0e-05" iyy="1e-05" izz="1e-05" ixy="0.0" iyz="0.0" ixz="-0.0"/>
   </inertial>
   <visual>
-    <origin xyz="-0.565819 -0.244976 -0.020398" rpy="0 0 0"/>
+    <origin xyz="0.020398 -0.244976 -0.565819" rpy="0 -1.57079632679 0"/>
     <geometry>
       <mesh filename="package://eternalmorph_description/meshes/sag_arka_pervane_1.stl" scale="0.001 0.001 0.001"/>
@@ -404,5 +404,5 @@
   </visual>
   <collision>
-    <origin xyz="-0.565819 -0.244976 -0.020398" rpy="0 0 0"/>
+    <origin xyz="0.020398 -0.244976 -0.565819" rpy="0 -1.57079632679 0"/>
     <geometry>
       <mesh filename="package://eternalmorph_description/meshes/sag_arka_pervane_1.stl" scale="0.001 0.001 0.001"/>
@@ -412,10 +412,10 @@
 <link name="sag_on_pervane_1">
   <inertial>
-    <origin xyz="0.0026102891123487293 3.06068145106142e-07 6.712215920232079e-07" rpy="0 0 0"/>
+    <origin xyz="-6.7122159e-07 3.0606815e-07 0.0026102891" rpy="0 -1.57079632679 0"/>
     <mass value="0.027453359988130525"/>
     <inertia ixx="1.0e-05" iyy="1e-05" izz="1e-05" ixy="-0.0" iyz="0.0" ixz="0.0"/>
   </inertial>
   <visual>
-    <origin xyz="-0.565819 0.374976 -0.020386" rpy="0 0 0"/>
+    <origin xyz="0.020386 0.374976 -0.565819" rpy="0 -1.57079632679 0"/>
     <geometry>
       <mesh filename="package://eternalmorph_description/meshes/sag_on_pervane_1.stl" scale="0.001 0.001 0.001"/>
@@ -424,5 +424,5 @@
   </visual>
   <collision>
-    <origin xyz="-0.565819 0.374976 -0.020386" rpy="0 0 0"/>
+    <origin xyz="0.020386 0.374976 -0.565819" rpy="0 -1.57079632679 0"/>
     <geometry>
       <mesh filename="package://eternalmorph_description/meshes/sag_on_pervane_1.stl" scale="0.001 0.001 0.001"/>
@@ -499,26 +499,26 @@
 </joint>
 <joint name="sol_on_pervane_joint" type="continuous">
-  <origin xyz="-0.019 0.0 0.0" rpy="0 0 0"/>
+  <origin xyz="-0.019 0.0 0.0" rpy="0 -1.57079632679 0"/>
   <parent link="sol_on_teker_1"/>
   <child link="sol_on_pervane_1"/>
-  <axis xyz="-1.0 0.0 0.0"/>
+  <axis xyz="0.0 0.0 1.0"/>
 </joint>
 <joint name="sol_arka_pervane_joint" type="continuous">
-  <origin xyz="-0.019 0.0 -0.000392" rpy="0 0 0"/>
+  <origin xyz="-0.019 0.0 -0.000392" rpy="0 -1.57079632679 0"/>
   <parent link="sol_arka_teker_1"/>
   <child link="sol_arka_pervane_1"/>
-  <axis xyz="-1.0 0.0 0.0"/>
+  <axis xyz="0.0 0.0 1.0"/>
 </joint>
 <joint name="sag_on_pervane_joint" type="continuous">
-  <origin xyz="0.019 0.0 0.000392" rpy="0 0 0"/>
+  <origin xyz="0.019 0.0 0.000392" rpy="0 1.57079632679 0"/>
   <parent link="sag_on_teker_1"/>
   <child link="sag_on_pervane_1"/>
-  <axis xyz="1.0 0.0 0.0"/>
+  <axis xyz="0.0 0.0 1.0"/>
 </joint>
 <joint name="sag_arka_pervane_joint" type="continuous">
-  <origin xyz="0.019 0.0 0.000392" rpy="0 0 0"/>
+  <origin xyz="0.019 0.0 0.000392" rpy="0 1.57079632679 0"/>
   <parent link="sag_arka_teker_1"/>
   <child link="sag_arka_pervane_1"/>
-  <axis xyz="1.0 0.0 0.0"/>
+  <axis xyz="0.0 0.0 1.0"/>
 </joint>
 <joint name="bacak_fixed_joint" type="fixed">

Commit message: Added camera

File: morphobot-ros2/eternalmorph_description/urdf/eternalmorph.xacro (robot description, xacro)
@@ -591,3 +591,35 @@
   <dynamics damping="2.0" friction="0.2"/>
 </joint>
+<link name="camera_1">
+    <inertial>
+      <origin xyz="7.9669377317515e-08 0.007701579533281336 0.019385691102944518" rpy="0 0 0"/>
+      <mass value="0.0441171047069775"/>
+      <inertia ixx="6e-06" iyy="5e-06" izz="5e-06" ixy="0.0" iyz="0.0" ixz="-0.0"/>
+    </inertial>
+    <visual>
+      <origin xyz="-0.42 -0.1 -0.01" rpy="0 0 0"/>
+      <geometry>
+        <mesh filename="package://eternalmorph_description/meshes/camera_1.stl" scale="0.001 0.001 0.001"/>
+      </geometry>
+      <material name="silver"/>
+    </visual>
+    <collision>
+      <origin xyz="-0.42 -0.1 -0.01" rpy="0 0 0"/>
+      <geometry>
+        <mesh filename="package://eternalmorph_description/meshes/camera_1.stl" scale="0.001 0.001 0.001"/>
+      </geometry>
+    </collision>
+  </link>
+  <joint name="camera_joint" type="fixed">
+    <origin xyz="0.42 0.1 0.01" rpy="0 0 0"/>
+    <parent link="base_link"/>
+    <child link="camera_1"/>
+  </joint>
+  <!-- Optical frame for ROS camera conventions (Z forward, X right, Y down) -->
+  <link name="camera_1_optical_frame"/>
+  <joint name="camera_1_optical_joint" type="fixed">
+    <origin xyz="0 0.025 0.02" rpy="-1.5707963 0 0"/>
+    <parent link="camera_1"/>
+    <child link="camera_1_optical_frame"/>
+  </joint>
 </robot>

Commit message: add closed-loop PID attitude controller and IMU sensor integration

File: morphobot-ros2/eternalmorph_description/urdf/eternalmorph.xacro (robot description, xacro)
@@ -623,3 +623,16 @@
     <child link="camera_1_optical_frame"/>
   </joint>
+  <!-- IMU link placed at the robot's actual Center of Mass (CoM) -->
+  <link name="imu_link">
+    <inertial>
+      <mass value="0.001"/>
+      <origin xyz="0 0 0" rpy="0 0 0"/>
+      <inertia ixx="1e-07" iyy="1e-07" izz="1e-07" ixy="0" ixz="0" iyz="0"/>
+    </inertial>
+  </link>
+  <joint name="imu_joint" type="fixed">
+    <origin xyz="0.4200 -0.0644 0.0236" rpy="0 0 0"/>
+    <parent link="base_link"/>
+    <child link="imu_link"/>
+  </joint>
 </robot>

Commit message: Added ground teleop and ros2control

File: morphobot-ros2/eternalmorph_description/urdf/eternalmorph.xacro (robot description, xacro)
@@ -636,3 +636,47 @@
     <child link="imu_link"/>
   </joint>
+  <!-- ===== ros2_control HARDWARE TANIMI (rover_ws ile birebir aynı mimari) ===== -->
+  <ros2_control name="GazeboSystem" type="system">
+    <hardware>
+      <plugin>gz_ros2_control/GazeboSimSystem</plugin>
+    </hardware>
+    <joint name="sol_on_teker">
+      <command_interface name="velocity">
+        <param name="min">-20.0</param>
+        <param name="max">20.0</param>
+      </command_interface>
+      <state_interface name="position"/>
+      <state_interface name="velocity"/>
+    </joint>
+    <joint name="sag_on_teker">
+      <command_interface name="velocity">
+        <param name="min">-20.0</param>
+        <param name="max">20.0</param>
+      </command_interface>
+      <state_interface name="position"/>
+      <state_interface name="velocity"/>
+    </joint>
+    <joint name="sol_arka_teker">
+      <command_interface name="velocity">
+        <param name="min">-20.0</param>
+        <param name="max">20.0</param>
+      </command_interface>
+      <state_interface name="position"/>
+      <state_interface name="velocity"/>
+    </joint>
+    <joint name="sag_arka_teker">
+      <command_interface name="velocity">
+        <param name="min">-20.0</param>
+        <param name="max">20.0</param>
+      </command_interface>
+      <state_interface name="position"/>
+      <state_interface name="velocity"/>
+    </joint>
+  </ros2_control>
+  <!-- ===== GAZEBO ROS2 CONTROL PLUGIN ===== -->
+  <gazebo>
+    <plugin filename="gz_ros2_control-system" name="gz_ros2_control::GazeboSimROS2ControlPlugin">
+      <parameters>$(find eternalmorph_description)/config/controllers.yaml</parameters>
+    </plugin>
+  </gazebo>
 </robot>
